File: (OLD) solenoid-control-board.kicad_sch (KiCad schematic)
At the start: 39 parts, among them J1 505578-0671, J2 505578-0671, J3 SM04B-GHS-TB, J4 XT30PW-M30.G.Y1, J5 XT30PW-M30.G.Y1, M1 CSD16323Q3, M2 CSD16323Q3, M3 CSD16323Q3, M4 CSD16323Q3, M5 CSD16323Q3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

Commit message: Working on layout
Parts:
- removed H1, H2, H3: ~, Downloaded:HDR-TH_6P-P2.54-V-M-R2-C3-S2.54-2, symbol Downloaded:HX PZ2.54-2X3P ZZ
- added U1, U2, U3, U4, U5, U6: L102011MS02Q, Downloaded:L102011MS02Q_CNK, symbol solenoid_control_board:L102011MS02Q
- M1, M2, M3, M4, M5, M6: footprint Downloaded:TRANS_CSD17308Q3 -> Downloaded:DQG0008A
Connections:
- net +12V: now also U1.2, U2.2, U3.2, U4.2, U5.2, U6.2
- net +6V: now also U1.3, U2.3, U3.3, U4.3, U5.3, U6.3
- net GND: no longer J4.3, J4.4, J5.3, J5.4
- net SOL_1_PWR: now also J1.1; no longer J1.5
- net SOL_3_PWR: now also J1.5; no longer J1.1
- net SOL_4_PWR: now also J2.1; no longer J2.5
- net SOL_6_PWR: now also J2.5; no longer J2.1
- net SRC_1: no longer names the net of M1.2, R1.1
- net SRC_1: now also U1.1
- net SRC_2: no longer names the net of M2.2, R3.1
- net SRC_2: now also U2.1
- net SRC_3: no longer names the net of M3.2, R5.1
- net SRC_3: now also U3.1
- net SRC_4: no longer names the net of M4.2, R7.1
- net SRC_4: now also U4.1
- net SRC_5: no longer names the net of M5.2, R9.1
- net SRC_5: now also U5.1
- net SRC_6: no longer names the net of M6.2, R11.1
- net SRC_6: now also U6.1
Other:
- note removed: "Pin Headers"
- moved on the sheet: D1, D10, D11, D12, D2, D3, D4, D5, D6, D7, D8, D9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
