File: solenoid-control-board.kicad_sch (KiCad schematic)
At the start: 39 parts, among them J1 505578-0671, J2 505578-0671, J3 SM04B-GHS-TB, J4 XT30PW-M30.G.Y1, J5 XT30PW-M30.G.Y1, M1 CSD16323Q3, M2 CSD16323Q3, M3 CSD16323Q3, M4 CSD16323Q3, M5 CSD16323Q3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

Commit message: Finished almost everything
Connections:
- net +12V: now also H1.1, H1.2, H2.1, H2.2, H3.1, H3.2; no longer H1.5, H1.6, H2.5, H2.6, H3.5, H3.6
- net +6V: now also H1.5, H1.6, H2.5, H2.6, H3.5, H3.6; no longer H1.1, H1.2, H2.1, H2.2, H3.1, H3.2
- net GND: now also J1.1, J1.3, J1.5, J2.1, J2.3, J2.5; no longer J1.2, J1.4, J1.6, J2.2, J2.4, J2.6
- net SOL_1_PWR: now also J1.6; no longer J1.5
- net SOL_2_PWR: now also J1.4; no longer J1.3
- net SOL_3_PWR: now also J1.2; no longer J1.1
- net SOL_4_PWR: now also J2.6; no longer J2.5
- net SOL_5_PWR: now also J2.4; no longer J2.3
- net SOL_6_PWR: now also J2.2; no longer J2.1
- net SRC_1: now also H1.4; no longer H1.3
- net SRC_2: now also H1.3; no longer H1.4
- net SRC_3: now also H2.4; no longer H2.3
- net SRC_4: now also H2.3; no longer H2.4
- net SRC_5: now also H3.4; no longer H3.3
- net SRC_6: now also H3.3; no longer H3.4
Other:
- moved on the sheet: H1, H2, H3

Commit message: Finished layout, need to simulate
Connections:
- net GND: now also J1.MP1, J1.MP2, J2.MP1, J2.MP2, J3.5, J3.6
