File: solenoid-control-board.kicad_sch (KiCad schematic)
At the start: 39 parts, among them J1 505578-0671, J2 505578-0671, J3 SM04B-GHS-TB, J4 XT30PW-M30.G.Y1, J5 XT30PW-M30.G.Y1, M1 CSD16323Q3, M2 CSD16323Q3, M3 CSD16323Q3, M4 CSD16323Q3, M5 CSD16323Q3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

Commit message: Generated BOM
Parts:
- D1, D11, D3, D5, D7, D9: footprint Downloaded:LED0603-R-RD_ORANGE -> solenoid-control-board:LED0603-R-RD_ORANGE; LCSC (none) -> C434425
- D10, D12, D2, D4, D6, D8: footprint Downloaded:LED0603-R-RD_GREEN -> solenoid-control-board:LED0603-R-RD_GREEN; LCSC (none) -> C19712532
- H1, H2, H3: value ~ -> HX PZ2.54-2x3P ZZ; footprint Downloaded:HDR-TH_6P-P2.54-V-M-R2-C3-S2.54-2 -> solenoid-control-board:HDR-TH_6P-P2.54-V-M-R2-C3-S2.54-2; LCSC (none) -> C32713276
- J1, J2: footprint Downloaded:5055780671 -> solenoid-control-board:5055780671; LCSC (none) -> C5362280
- J3: footprint Downloaded:CONN_SM04B-GHS-TB_JST -> solenoid-control-board:CONN_SM04B-GHS-TB_JST; LCSC (none) -> C189895
- J4, J5: value XT30PW-M30.G.Y1 -> XT30PW-M30.G.Y; footprint Downloaded:CONN-TH_XT30PW-M -> solenoid-control-board:CONN-TH_XT30PW-M; LCSC (none) -> C431092
- M1, M2, M3, M4, M5, M6: footprint Downloaded:TRANS_CSD17308Q3 -> solenoid-control-board:TRANS_CSD17308Q3; LCSC (none) -> C248610
- R1, R10, R11, R12, R2, R3, R4, R5, R6, R7, R8, R9: value 4.7kΩ -> R; footprint Downloaded:RESC1607X60N -> solenoid-control-board:RESC1607X60N; LCSC (none) -> C99782
- U7: footprint Downloaded:PW16 -> solenoid-control-board:PW16; LCSC (none) -> C133803
